Commit message: Latest Practice Mazes with Beacons

File: urdf/turtlebot3_waffle.urdf (robot description, URDF)
Before this commit: robot turtlebot3_waffle, 13 links, 12 joints
Links:
- removed link realsense_depth_frame
- removed link realsense_link
- added link camera_depth_frame
- added link camera_link; collision box size=0.012 0.132 0.020; visual mesh filename=package://turtlebot3_gazebo/models/turtlebot3_common/meshes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
- link base_link: geometry collision box size=0.266 0.266 0.094; visual mesh filename=package://turtlebot3_gazebo/models/turtlebot3_common/meshes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 scale=0.001 0.001 0.001
- link base_scan: geometry collision cylinder length=0.0315 radius=0.055; visual mesh filename=package://turtlebot3_gazebo/models/turtlebot3_common/meshes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 scale=0.001 0.001 0.001
- link wheel_left_link: geometry collision cylinder length=0.018 radius=0.033; visual mesh filename=package://turtlebot3_gazebo/models/turtlebot3_common/meshes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 scale=0.001 0.001 0.001
- link wheel_right_link: geometry collision cylinder length=0.018 radius=0.033; visual mesh filename=package://turtlebot3_gazebo/models/turtlebot3_common/meshes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 scale=0.001 0.001 0.001
Joints:
- removed joint realsense_depth_joint
- added joint camera_depth_joint: type fixed, parent camera_link, child camera_depth_frame, origin xyz=0.005 0.028 0.013 rpy=0 0 0
- joint camera_depth_optical_joint: parent realsense_depth_frame -> camera_depth_frame
- joint camera_joint: child realsense_link -> camera_link
- joint camera_rgb_joint: origin xyz=0.005 0.018 0.013 rpy=-1.57 0 -1.57 -> xyz=0.005 0.018 0.013 rpy=0 0 0; parent realsense_link -> camera_link
